File: oya45.kicad_pcb (KiCad board)
At the start: 2 copper layers, 190.5 x 95.2 mm, 106 parts, among them U1 ProMicro

Commit message: final
finalized bottom row and pcb
Routing:
- net col8: track 159.1 -> 161.9 mm
- net col0: track 165.2 -> 166.4 mm
Changed lines of the file:
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@@
     (thickness 1.6)
     (drawings 8)
-    (tracks 286)
+    (tracks 293)
     (zones 0)
     (modules 106)
@@
   (segment (start 216.535 33.02) (end 212.43625 37.11875) (width 0.254) (layer F.Cu) (net 50))
   (segment (start 60.96 54.61) (end 60.96 92.71) (width 0.254) (layer B.Cu) (net 51))
-  (segment (start 60.96 92.71) (end 60.96 111.76) (width 0.254) (layer B.Cu) (net 51))
   (segment (start 125.488701 46.596299) (end 126.365 45.72) (width 0.254) (layer B.Cu) (net 51))
   (segment (start 124.00599 48.07901) (end 125.488701 46.596299) (width 0.254) (layer B.Cu) (net 51))
@@
   (segment (start 60.96 54.61) (end 67.49099 48.07901) (width 0.254) (layer B.Cu) (net 51))
   (segment (start 62.55099 111.76) (end 75.2475 111.76) (width 0.254) (layer B.Cu) (net 51))
-  (segment (start 60.96 111.76) (end 62.55099 111.76) (width 0.254) (layer B.Cu) (net 51))
   (segment (start 68.41776 116.84) (end 70.00875 116.84) (width 0.254) (layer B.Cu) (net 51))
   (segment (start 56.255066 116.84) (end 68.41776 116.84) (width 0.254) (layer B.Cu) (net 51))
@@
   (segment (start 56.255066 111.76) (end 54.829099 113.185967) (width 0.254) (layer B.Cu) (net 51))
   (segment (start 60.96 111.76) (end 56.255066 111.76) (width 0.254) (layer B.Cu) (net 51))
+  (segment (start 62.55099 111.76) (end 60.96 111.76) (width 0.254) (layer B.Cu) (net 51))
+  (segment (start 63.205751 111.105239) (end 62.55099 111.76) (width 0.254) (layer B.Cu) (net 51))
+  (segment (start 63.205751 108.523039) (end 63.205751 111.105239) (width 0.254) (layer B.Cu) (net 51))
+  (segment (start 60.96 106.277288) (end 63.205751 108.523039) (width 0.254) (layer B.Cu) (net 51))
+  (segment (start 60.96 92.71) (end 60.96 106.277288) (width 0.254) (layer B.Cu) (net 51))
   (segment (start 80.01 54.61) (end 80.01 111.76) (width 0.254) (layer B.Cu) (net 52))
   (segment (start 128.028701 46.596299) (end 128.905 45.72) (width 0.254) (layer B.Cu) (net 52))
@@
   (segment (start 194.31 108.044834) (end 194.31 111.76) (width 0.254) (layer B.Cu) (net 58))
   (segment (start 195.195801 107.159033) (end 194.31 108.044834) (width 0.254) (layer B.Cu) (net 58))
-  (segment (start 213.36 54.61) (end 213.36 111.76) (width 0.254) (layer B.Cu) (net 59))
   (segment (start 203.835 45.085) (end 203.835 35.56) (width 0.254) (layer B.Cu) (net 59))
   (segment (start 213.36 54.61) (end 203.835 45.085) (width 0.254) (layer B.Cu) (net 59))
@@
   (segment (start 197.64375 29.36875) (end 134.337136 29.36875) (width 0.254) (layer B.Cu) (net 59))
   (segment (start 203.835 35.56) (end 197.64375 29.36875) (width 0.254) (layer B.Cu) (net 59))
+  (segment (start 214.95099 111.76) (end 213.36 111.76) (width 0.254) (layer B.Cu) (net 59))
+  (segment (start 215.605751 111.105239) (end 214.95099 111.76) (width 0.254) (layer B.Cu) (net 59))
+  (segment (start 215.605751 108.523039) (end 215.605751 111.105239) (width 0.254) (layer B.Cu) (net 59))
+  (segment (start 213.36 106.277288) (end 215.605751 108.523039) (width 0.254) (layer B.Cu) (net 59))
+  (segment (start 213.36 54.61) (end 213.36 106.277288) (width 0.254) (layer B.Cu) (net 59))
   (segment (start 232.41 54.61) (end 232.41 111.76) (width 0.254) (layer B.Cu) (net 60))
   (segment (start 222.885 45.085) (end 222.885 35.56) (width 0.254) (layer B.Cu) (net 60))

Commit message: added callmevroyasumi soldermask
Parts:
- added G***: LOGO, soldermask:callmevroyasumi, B.Cu at (73.8, 38.1)
